File: GRPv1.2RasToNew/IO:Sensor Board.kicad_pcb (KiCad board)
At the start: 2 copper layers, 70 x 80 mm, 20 parts, among them J1 B3B-XH-A, J3 B6B-XH-A, J4 B2B-XH-A, U1 BMP581, U3 TPS79333-EP, U4 ICM-20948, U5 TPS79318-EP

Commit message: teensy modification
Parts:
- removed Module1: ComputeModule4-CM4, CM4IO:Raspberry-Pi-4-Compute-Module
- added U6: Teensy4.1, modFiles:Teensy41, F.Cu at (172.3, 102.1)
- moved J1 67.3 mm to (193.5, 116.0), turned to -90 degrees
- moved J4 64.5 mm to (193.5, 81.5), turned to 90 degrees
- moved J3 62.0 mm to (193.5, 93.5), turned to -90 degrees
- moved G*** 45.1 mm to (108.5, 85.0)
- moved C11 9.46 mm to (152.0, 111.0), turned to -90 degrees
- moved C13 8.56 mm to (148.5, 106.5), turned to 135 degrees
- moved C5 5.35 mm to (137.4, 117.7), turned to -45 degrees
- moved C2 5.27 mm to (151.4, 80.9)
- moved C3 5.27 mm to (152.0, 83.9)
- moved U1 5.27 mm to (153.8, 81.2)
- moved C4 4.98 mm to (138.5, 92.0)
- moved C6 4.98 mm to (140.1, 93.6)
- moved U5 4.98 mm to (141.9, 90.0)
- moved C8 4.98 mm to (143.8, 88.1)
- moved C12 3.39 mm to (151.7, 102.2), turned to 45 degrees
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Routing:
- net GND: track 184.8 -> 44.8 mm, vias 34 -> 17
- net ICM_CLK: track 31.5 -> 93.1 mm, vias 0 -> 4
- net PYRO_2: track 79.3 -> 17.8 mm, vias 2 -> 0
- net PYRO_5: track 76.8 -> 16.8 mm, vias 2 -> 0
- net SERVO_4: track 74.8 -> 16.8 mm, vias 2 -> 0
- net PYRO_4: track 73.2 -> 16.8 mm, vias 2 -> 0
- net FSYNC: track 50.0 -> 0.00 mm, vias 2 -> 0
- net PYRO_3: track 60.9 -> 17.8 mm, vias 2 -> 0
- net SERVO_3: track 59.1 -> 16.8 mm, vias 2 -> 0
- net BMP_MOSI: track 21.3 -> 62.0 mm, vias 0 -> 2
- net ICM_CS: track 20.9 -> 58.5 mm
- net SERVO_2: track 53.5 -> 18.9 mm, vias 2 -> 0
- net PYRO_1: track 51.9 -> 17.8 mm, vias 2 -> 0
- net +5V: track 92.4 -> 125.4 mm, vias 2 -> 0
- net ICM_INT: track 32.0 -> 0.00 mm, vias 2 -> 0
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Other:
- board size 70 x 80 mm -> 70 x 70 mm

Commit message: esp switch 1
Parts:
- removed U6: Teensy4.1, modFiles:Teensy41
- added C10: 10uF, Capacitors:C_0805_2012Metric_Pad1.18x1.45mm_HandSolder, F.Cu at (188.5, 76.5)
- added C14: 10uF, Capacitors:C_0805_2012Metric_Pad1.18x1.45mm_HandSolder, F.Cu at (177.5, 69.0)
- added C15: 100uF, Capacitors:C_0805_2012Metric_Pad1.18x1.45mm_HandSolder, F.Cu at (178.0, 80.5)
- added C9: 100uF, Capacitors:C_0805_2012Metric_Pad1.18x1.45mm_HandSolder, F.Cu at (186.0, 88.0)
- added J2: B3B-XH-A, B3B:CONN_B3B-XH-A_JST, F.Cu at (146.5, 71.0)
- added J5: B3B-XH-A, B3B:CONN_B3B-XH-A_JST, F.Cu at (135.0, 77.0)
- added JP1: Jumper_2_Open, Jumper:SolderJumper-2_P1.3mm_Open_RoundedPad1.0x1.5mm, F.Cu at (196.5, 87.2)
- added JP2: Jumper_2_Open, Jumper:SolderJumper-2_P1.3mm_Open_RoundedPad1.0x1.5mm, F.Cu at (196.5, 78.3)
- added JP3: Jumper_2_Open, Jumper:SolderJumper-2_P1.3mm_Open_RoundedPad1.0x1.5mm, F.Cu at (185.0, 93.0)
- added P1: 282837-2, ScrewTerminal:CUI_TB002-500-02BE, F.Cu at (194.7, 118.5)
- added P2: 282837-2, ScrewTerminal:CUI_TB002-500-02BE, F.Cu at (194.5, 107.5)
- added P3: 282837-2, ScrewTerminal:CUI_TB002-500-02BE, F.Cu at (194.5, 96.5)
- added Q1: DMN3023L-7, FETS:SOT96P240X100-3N, F.Cu at (188.5, 126.5)
- added Q2: DMN3023L-7, FETS:SOT96P240X100-3N, F.Cu at (188.5, 117.4)
- added Q3: DMN3023L-7, FETS:SOT96P240X100-3N, F.Cu at (188.5, 107.4)
- added R1: 1k, Resistor:R_0805_2012Metric_Pad1.20x1.40mm_HandSolder, F.Cu at (185.5, 126.5)
- added R2: 470, Resistor:R_0805_2012Metric_Pad1.20x1.40mm_HandSolder, F.Cu at (186.5, 129.5)
- added R3: 1k, Resistor:R_0805_2012Metric_Pad1.20x1.40mm_HandSolder, F.Cu at (185.5, 117.5)
- added R4: 470, Resistor:R_0805_2012Metric_Pad1.20x1.40mm_HandSolder, F.Cu at (186.5, 120.5)
- added R5: 1k, Resistor:R_0805_2012Metric_Pad1.20x1.40mm_HandSolder, F.Cu at (185.5, 107.4)
- added R6: 470, Resistor:R_0805_2012Metric_Pad1.20x1.40mm_HandSolder, F.Cu at (186.5, 110.4)
- added U10: XT30UPB-M, XTConnectors:XT30UPB-M, F.Cu at (167.0, 71.0)
- added U2: DEVKIT_V1_ESP32-WROOM-32, esp32wroom:MODULE_DEVKIT_V1_ESP32-WROOM-32, F.Cu at (159.9, 106.7)
- added U7: LD1117S50CTR, LD1117S50CTRlib:LD1117S50CTR, F.Cu at (189.5, 82.5)
- added U8: XT30UPB-M, XTConnectors:XT30UPB-M, F.Cu at (156.0, 71.0)
- added U9: LD1117S50CTR, LD1117S50CTRlib:LD1117S50CTR, F.Cu at (179.0, 74.5)
- C1, C11, C12, C13, C2, C3, C4, C5, C6, C7, C8: footprint Capacitor_SMD:C_0805_2012Metric_Pad1.18x1.45mm_HandSolder -> Capacitors:C_0805_2012Metric_Pad1.18x1.45mm_HandSolder
- J1: footprint Connector_JST:JST_XH_B3B-XH-A_1x03_P2.50mm_Vertical -> B3B:CONN_B3B-XH-A_JST
- moved J3 58.7 mm to (135.0, 88.5)
- moved G*** 51.8 mm to (153.3, 111.1)
- moved J1 51.6 mm to (146.1, 95.6), turned to 45 degrees
- moved C7 35.3 mm to (145.8, 78.4), turned to -22.5 degrees
- moved U3 34.8 mm to (144.5, 81.1), turned to -22.5 degrees
- moved C5 34.3 mm to (143.5, 83.9), turned to -22.5 degrees
- moved C13 33.6 mm to (173.5, 129.0), turned to -135 degrees
- moved C1 33.6 mm to (141.3, 78.1), turned to -67.5 degrees
- moved C11 29.8 mm to (178.0, 125.5), turned to 0 degrees
- moved C12 29.4 mm to (169.2, 125.8), turned to 135 degrees
- moved U4 27.2 mm to (173.0, 124.5), turned to 0 degrees
- moved U5 18.6 mm to (156.5, 78.4)
- moved C4 18.6 mm to (153.1, 80.4)
- moved C6 18.6 mm to (154.7, 82.0)
- moved C8 18.6 mm to (158.4, 76.5)
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Connections:
- net +5V renamed +5V_b
Routing:
- net +12V: track 0.00 -> 109.1 mm, vias 0 -> 1
- net +3.3V_b: track 56.9 -> 151.4 mm, vias 2 -> 4
- net +1.8V: track 23.8 -> 110.3 mm, vias 0 -> 2
- net ICM_CLK: track 93.1 -> 11.0 mm, vias 4 -> 0
- net +5V_b: track 125.4 -> 68.4 mm
- net BMP_CLK: track 56.2 -> 11.4 mm, vias 4 -> 0
- net SERVO_1: track 18.9 -> 61.6 mm
- net SERVO_2: track 18.9 -> 60.2 mm
- net SERVO_3: track 16.8 -> 57.4 mm
- net GND: track 44.8 -> 83.9 mm, vias 17 -> 23
- net SERVO_4: track 16.8 -> 55.2 mm
- net PYRO_4: track 16.8 -> 53.1 mm
- net PYRO_5: track 16.8 -> 51.3 mm
- net SERVO_6: track 0.00 -> 31.9 mm
- net BMP_MOSI: track 62.0 -> 30.7 mm, vias 2 -> 1
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- added copper zone on In1.Cu, net GND
- added copper zone on In2.Cu, net GND
- removed copper zone on B.Cu, net GND
Other:
- copper layers 2 -> 4

Commit message: save 2
Parts:
- moved G*** 3.88 mm to (157.1, 110.3)
- moved R3 0.98 mm to (184.8, 116.9)
- moved R4 0.98 mm to (185.8, 119.9)
- moved Q2 0.98 mm to (187.8, 116.8)
- moved Q3 0.93 mm to (187.5, 107.3)
- moved R5 0.93 mm to (184.5, 107.3)
- moved R6 0.93 mm to (185.5, 110.3)
- moved J2 0.33 mm to (146.5, 71.3)
- moved P1 0.20 mm to (194.5, 118.5)
Routing:
- net +5V_b: track 68.4 -> 109.4 mm, vias 0 -> 1
- net +12V: track 109.1 -> 124.1 mm, vias 1 -> 2
- net +5V_a: track 13.4 -> 21.1 mm
- net +1.8V: track 110.3 -> 108.7 mm
- net PYRO_7: track 22.2 -> 21.7 mm
- net BMP_CS: track 17.8 -> 18.3 mm
- net GND: vias 23 -> 24
