File: GRPv1.2RasToNew/IO:Sensor Board.kicad_pcb (KiCad board)
At the start: 4 copper layers, 70 x 70 mm, 45 parts, among them J1 B3B-XH-A, J2 B3B-XH-A, J3 B6B-XH-A, J4 B2B-XH-A, J5 B3B-XH-A, P1 282837-2, P2 282837-2, P3 282837-2, Q1 DMN3023L-7, Q2 DMN3023L-7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

Commit message: checkoff with pwm
Parts:
- added J6: B3B-XH-A, NewJST:CONN_B3B-XH-A_JST, F.Cu at (160.3, 81.7)
- moved U5 51.6 mm to (162.7, 129.7)
- moved C8 51.6 mm to (164.6, 127.7)
- moved C4 51.6 mm to (159.4, 131.6)
- moved C6 51.6 mm to (161.0, 133.2)
Connections:
- U2 pad 26: unconnected-(U2-IO4-Pad26) -> SERVO_7
Routing:
- net +1.8V: track 108.7 -> 12.6 mm, vias 2 -> 0
- net +5V_b: track 109.4 -> 204.6 mm, vias 1 -> 3
- net SERVO_7: track 0.00 -> 12.3 mm
- net +3.3V_b: track 151.4 -> 147.5 mm
